File: spot_welder/spot_welder.kicad_pcb (KiCad board)
At the start: 2 copper layers, 93.7 x 117.2 mm, 93 parts, among them J1 Trigger, J2 Conn_SWD, J3 External_Power, Q1 NX3020NAKW, Q2 HY4903B6, Q3 HY4903B6, Q4 HY4903B6, Q5 HY4903B6, Q6 HY4903B6, Q7 HY4903B6, U1 STM32F103C8Tx, U2 SN74LVC1G123DCT, U3 LM2575-ADJ, U4 IRS44273LTRPBF, U5 AMS1117-3.3, U6 RC1602A

Commit message: code
Parts:
- added REF**: BUS_BAR_BOTTOM, spot_welder:BUS_BAR_BOTTOM, B.Cu at (99.2, 122.4)
- added REF**: BUS_BAR, spot_welder:BUS_BAR_TOP, B.Cu at (89.6, 89.6)
- C12, R7, R8: moved to F.Cu
- U6: footprint Display:WC1602A -> spot_welder:RC1602A
- moved C11 72.0 mm to (51.2, 126.4)
- moved C14 69.8 mm to (54.4, 123.6)
- moved R9 69.7 mm to (51.2, 123.6)
- moved R6 68.2 mm to (54.4, 126.4)
- moved R16 49.8 mm to (109.3, 134.2)
- moved R12 49.5 mm to (105.1, 134.2)
- moved R13 47.7 mm to (105.1, 137.1), turned to 180 degrees
- moved R10 46.8 mm to (100.8, 134.2)
- moved D9 40.3 mm to (109.3, 140.2)
- moved R11 38.9 mm to (100.8, 137.1), turned to 180 degrees
- moved C20 38.6 mm to (109.3, 143.3)
- moved R17 38.5 mm to (109.3, 137.1), turned to 180 degrees
- moved D7 38.1 mm to (105.1, 140.2)
- moved C12 35.6 mm to (83.8, 151.8), turned to 180 degrees
- moved D5 34.0 mm to (100.8, 140.2)
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Routing:
- net VEXT+: track 0.00 -> 5.31 mm

Commit message: migrate to kicad7
Other:
- net class Default removed
