File: spot_welder/power.kicad_sch (KiCad schematic)
At the start: 61 parts, among them J3 External_Power, Q2 HY4903B6, Q3 HY4903B6, Q4 HY4903B6, Q5 HY4903B6, Q6 HY4903B6, Q7 HY4903B6, U2 SN74LVC1G123DCT, U3 LM2575-ADJ, U4 IRS44273LTRPBF, U5 AMS1117-3.3

Commit message: 1
Parts:
- removed U2: SN74LVC1G123DCT, Package_SO:SSOP-8_2.95x2.8mm_P0.65mm, symbol spot_welder:SN74LVC1G123DCT
- added U2: SN74LVC1G123DCT, Package_SO:SSOP-8_2.95x2.8mm_P0.65mm, symbol 74xGxx:74LVC1G123
- C13: PartNo CK1V101MCRE77 -> C141427
- C18: value 16V 2200uF -> 16V 2200u; footprint Capacitor_THT:C_Radial_D12.5mm_H20.0mm_P5.00mm -> Capacitor_SMD:CP_Elec_16x17.5; PartNo 16YXJ2200M12.5X20 -> C239248
- C19, C21: PartNo (none) -> C19666
- D10, D11, D12, D13, D16, D8: PartNo MM3Z18VCW -> C2926440
- D14: PartNo SMBJ36A -> C5331118
- D15: value nb -> nc(BZW50-68); PartNo BZW50-68 -> (none)
- D4: PartNo SS34 -> C8678
- D5, D7, D9: PartNo MM3Z4V7 -> C2856973
- D6: footprint spot_welder:D_SOD-123FL -> Diode_SMD:D_SOD-123F; PartNo LMBR340FT1G -> C475721
- FB2: PartNo 2506031017Y0 -> C64181
- J3: footprint spot_welder:CONN-5.0-2P -> Connector_Phoenix_MSTB:PhoenixContact_MSTBVA_2,5_2-G_1x02_P5.00mm_Vertical; PartNo DB126V-5.0-2P -> C395849
- JP1: PartNo (none) -> C49257
- L1: PartNo SMRH127-471M -> C10153
- Q2, Q3, Q4, Q5, Q6, Q7: PartNo HY4903B6 -> C133393
- U3: PartNo LM2575S-ADJ/TR -> C347407
- U4: PartNo IRS44273LTRPBF -> C126909
- U5: PartNo AMS1117-3.3 -> C5250992
Connections:
- net +10V: now also C16.1, U4.5 (VCC)
- net +3V3: now also C14.2, U2.2 (B), U2.8 (VCC); no longer C14.1, C16.1, U4.5 (VCC)
- net GND: now also C14.1, U2.4 (GND); no longer C14.2
- net SW_OFF: now also U2.3 (~{CLR})
- net SW_ON: now also U2.1 (~{A})
- net at U4.1 (IN): now also U2.5 (Q)
- net at C11.2: now also U2.6 (Cext)
- net at C11.1, R9.1: now also U2.7 (RCext)
Other:
- note added: "Pulse width t=T*R*C=0.9*4.7e5*1e-6=0.423s"
- moved on the sheet: C11, C14, R6, R9
