File: spot_welder/spot_welder.kicad_sch (KiCad schematic)
At the start: 27 parts, among them J1 Trigger, J2 Conn_SWD, Q1 NX3020NAKW, U1 STM32F103C8Tx, U6 RC1602A

Commit message: 1
Parts:
- removed C5: 10nF, Capacitor_SMD:C_0603_1608Metric, symbol Device:C
- removed D2: 1N4148, Diode_SMD:D_SOD-123, symbol Device:D
- removed Q1: NX3020NAKW, Package_TO_SOT_SMD:SOT-323_SC-70, symbol Device:Q_NMOS_DGS
- removed U1: STM32F103C8Tx, Package_QFP:LQFP-48-1EP_7x7mm_P0.5mm_EP3.6x3.6mm, symbol common:STM32F103C8Tx
- added Q1: 2N4401, Package_TO_SOT_SMD:SOT-23, symbol Device:Q_NPN_BEC
- added U1: STM32F103C8T6, Package_QFP:LQFP-48_7x7mm_P0.5mm, symbol MCU_ST_STM32F1:STM32F103C8Tx
- BZ1: value PS1240P02BT -> SFN-1407PA7.6; footprint spot_welder:BUZ-TH_BD12.5-P5.00-D0.9 -> Buzzer_Beeper:Buzzer_15x7.5RM7.6; PartNo PS1240P02BT -> C360603
- C3, C4: value 50V 1uF -> 1uF
- D1: value BZT52C4V7 -> MM3Z4V7; footprint Diode_SMD:D_SOD-123 -> Diode_SMD:D_SOD-323; PartNo BZT52C4V7 -> C2856973
- D3: value 1N4148 -> nc(1N4148WS); footprint Diode_SMD:D_SOD-123 -> Diode_SMD:D_SOD-323; PartNo 1N4148W -> C2128
- FB1: PartNo 2506031017Y0 -> C64181
- J1: footprint spot_welder:CONN-5.0-2P -> Connector_Phoenix_MSTB:PhoenixContact_MSTBVA_2,5_2-G_1x02_P5.00mm_Vertical; PartNo DB126V-5.0-2P -> C395849
- J2: footprint Connector_PinHeader_2.54mm:PinHeader_1x05_P2.54mm_Vertical -> Connector_PinHeader_2.54mm:PinHeader_1x06_P2.54mm_Vertical; symbol Connector_Generic:Conn_01x05 -> Connector_Generic:Conn_01x06; PartNo (none) -> DB126V-5.0-2P
- R4: value 220k -> 1k
- RV1: footprint Connector_PinHeader_2.54mm:PinHeader_1x03_P2.54mm_Vertical -> Potentiometer_THT:Potentiometer_Bourns_3386C_Horizontal; PartNo 3296W-1-104 -> C330448
- RV2: footprint spot_welder:EVM2GSX80B14 -> Potentiometer_SMD:Potentiometer_Bourns_3214J_Horizontal; PartNo EVM2GSX80B14 -> C719176
- U6: value RC1602A -> HS1602A; footprint spot_welder:RC1602A -> Connector_PinSocket_2.54mm:PinSocket_1x16_P2.54mm_Vertical; PartNo LCM1602K-NSW-BBW -> C5329588
Connections:
- net +10VS: now also U1.13 (PA3)
- net +3V3: now also U6.15 (A/VEE), U1.1 (VBAT), U1.24 (VDD), U1.36 (VDD), U1.48 (VDD); no longer U6.16 (K)
- net BUZZER: now also R4.1, U1.40 (PB4), U1.41 (PB5)
- net DIAL: now also U1.43 (PB7)
- net GND: now also J2.4 (Pin_4), U6.16 (K), Q1.2 (E), U1.20 (PB2), U1.23 (VSS), U1.35 (VSS), U1.47 (VSS), U1.5 (PD0), U1.6 (PD1), U1.8 (VSSA); no longer J2.3 (Pin_3), R4.2, U6.15 (A/VEE)
- net LED_D0: now also U1.27 (PB14)
- net LED_D1: now also U1.26 (PB13)
- net LED_D2: now also U1.25 (PB12)
- net LED_D3: now also U1.22 (PB11)
- net LED_D4: now also U1.21 (PB10)
- net LED_D5: now also U1.17 (PA7)
- net LED_D6: now also U1.16 (PA6)
- net LED_D7: now also U1.15 (PA5)
- net LED_E: now also U6.6 (E), U1.28 (PB15); no longer U6.4 (RS)
- net LED_RS: now also U6.4 (RS), U1.30 (PA9); no longer U6.6 (E)
- net LED_RW: now also U1.29 (PA8)
- net NRST: now also J2.6 (Pin_6), U1.7 (NRST); no longer J2.5 (Pin_5)
- net OUT+S: now also U1.11 (PA1)
- net OUT-S: now also U1.10 (PA0)
- net SWDIO: now also J2.5 (Pin_5), U1.34 (PA13); no longer J2.4 (Pin_4)
- net SW_OFF: now also U1.18 (PB0)
- net SW_ON: now also U1.19 (PB1)
- net TRIGGER: now also U1.39 (PB3)
- net VBAT+S: now also U1.12 (PA2)
- net VDDA: now also U1.9 (VDDA)
- net at R3.2: now also U1.44 (BOOT0)
- net at BZ1.2 (+), D3.2 (A): now also Q1.3 (C)
- net SWDCLK renamed RXD_SWDCLK
- net RXD_SWDCLK: now also U1.37 (PA14)
- new net: Q1.1 (B), R4.2
- new net TXD: J2.3 (Pin_3), U1.42 (PB6)
- no-connect marks 15 -> 10
Other:
- moved on the sheet: R4
